File: imu.kicad_sch (KiCad schematic)
At the start: 0 parts

Commit message: imu, motor esc schematics
Parts:
- added C7, C8: 100nF, Capacitor_SMD:C_0603_1608Metric_Pad1.08x0.95mm_HandSolder, symbol Device:C_Small
- added C9: 2.2nF, Capacitor_SMD:C_0603_1608Metric_Pad1.08x0.95mm_HandSolder, symbol Device:C_Small
- added R3: 10k, Resistor_SMD:R_0603_1608Metric_Pad0.98x0.95mm_HandSolder, symbol Device:R_Small_US
- added U2: MPU-6000, Sensor_Motion:InvenSense_QFN-24_4x4mm_P0.5mm, symbol Sensor_Motion:MPU-6000
Connections:
- new net: C9.1, U2.20 (CPOUT)
- new net: C7.1, U2.10 (REGOUT)
- new net +3V3: C8.2, R3.1, U2.13 (VDD)
- new net GND: C7.2, C8.1, C9.2, U2.11 (FSYNC), U2.18 (GND)
- new net IMU_CS: R3.2, U2.8 (~{CS})
- new net IMU_INT: U2.12 (INT)
- new net IMU_MISO: U2.9 (AD0/MISO)
- new net IMU_MOSI: U2.24 (SDA/MOSI)
- new net IMU_SCK: U2.23 (SCL/SCLK)
- no-connect marks 0 -> 3

Commit message: more esc schematics, refactoring, root schematic edits
Changed lines of the file:
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@@
 	)
 	(global_label "IMU_SCK"
-		(shape input)
+		(shape output)
 		(at 138.43 68.58 90)
 		(fields_autoplaced yes)
@@
 	)
 	(global_label "IMU_MOSI"
-		(shape input)
+		(shape output)
 		(at 143.51 68.58 90)
 		(fields_autoplaced yes)
@@
 	)
 	(global_label "IMU_CS"
-		(shape input)
+		(shape output)
 		(at 135.89 54.61 0)
 		(fields_autoplaced yes)
@@
 	)
 	(global_label "IMU_INT"
-		(shape input)
+		(shape output)
 		(at 143.51 107.95 180)
 		(fields_autoplaced yes)
@@
 	)
 	(global_label "IMU_MISO"
-		(shape input)
+		(shape output)
 		(at 140.97 68.58 90)
 		(fields_autoplaced yes)

Commit message: done?
Parts:
- removed C9: 2.2nF, Capacitor_SMD:C_0603_1608Metric_Pad1.08x0.95mm_HandSolder, symbol Device:C_Small
- removed U2: MPU-6000, Sensor_Motion:InvenSense_QFN-24_4x4mm_P0.5mm, symbol Sensor_Motion:MPU-6000
- added C44: 10nF, Capacitor_SMD:C_0603_1608Metric_Pad1.08x0.95mm_HandSolder, symbol Device:C_Small
- added C45: 2.2uF, Capacitor_SMD:C_0603_1608Metric_Pad1.08x0.95mm_HandSolder, symbol Device:C_Small
- added U9: ICM-20602, Package_LGA:LGA-16_3x3mm_P0.5mm, symbol Sensor_Motion:ICM-20602
- R3: footprint Resistor_SMD:R_0603_1608Metric_Pad0.98x0.95mm_HandSolder -> Resistor_SMD:R_0402_1005Metric_Pad0.72x0.64mm_HandSolder
Connections:
- net +3V3: now also C44.2, C45.2, U9.1 (VDDIO), U9.16 (VDD)
- net GND: now also C7.1, C44.1, C45.1, U9.10 (GND), U9.11 (GND), U9.12 (GND), U9.13 (GND), U9.15 (GND), U9.9 (GND); no longer C7.2
- net IMU_CS: now also U9.5 (~{CS})
- net IMU_INT: now also U9.6 (INT)
- net IMU_MISO: now also U9.4 (SAO/SD0)
- net IMU_MOSI: now also U9.3 (SDA/SDI)
- net IMU_SCK: now also U9.2 (SCL/SPC)
- new net: C7.2, U9.14 (REGOUT)
- no-connect marks 3 -> 1
