File: rc.kicad_sch (KiCad schematic)
At the start: 0 parts

Commit message: done?
Parts:
- added J15: Conn_01x04_Socket, Connector_PinSocket_1.00mm:PinSocket_1x04_P1.00mm_Vertical_SMD_Pin1Left, symbol Connector:Conn_01x04_Socket
Connections:
- new net +5V: J15.1 (Pin_1)
- new net CRSF_RX: J15.2 (Pin_2)
- new net CRSF_TX: J15.3 (Pin_3)
- new net GND: J15.4 (Pin_4)
