File: neodrone-v1.kicad_pcb (KiCad board)
At the start: 4 copper layers, 150 x 105 mm, 79 parts, among them J1 Conn_01x05_Socket, J10 SolderWirePad_1x01_SMD_3x6mm, J11 SolderWirePad_1x01_SMD_3x6mm, J12 SolderWirePad_1x01_SMD_3x6mm, J13 SolderWirePad_1x01_SMD_3x6mm, J14 Conn_01x02, J2 SolderWirePad_1x01_SMD_3x6mm, J3 SolderWirePad_1x01_SMD_3x6mm, J4 SolderWirePad_1x01_SMD_3x6mm, J5 SolderWirePad_1x01_SMD_3x6mm, J6 SolderWirePad_1x01_SMD_3x6mm, J7 SolderWirePad_1x01_SMD_3x6mm, J8 SolderWirePad_1x01_SMD_3x6mm, J9 SolderWirePad_1x01_SMD_3x6mm, M1 MountingHole_2.2mm_M2, M10 MountingHole_2.2mm_M2, M11 MountingHole_2.2mm_M2, M12 MountingHole_2.2mm_M2, M13 MountingHole_2.2mm_M2, M14 MountingHole_2.2mm_M2, M15 MountingHole_2.2mm_M2, M16 MountingHole_2.2mm_M2, M2 MountingHole_2.2mm_M2, M3 MountingHole_2.2mm_M2, M4 MountingHole_2.2mm_M2, M5 MountingHole_2.2mm_M2, M6 MountingHole_2.2mm_M2, M7 MountingHole_2.2mm_M2, M8 MountingHole_2.2mm_M2, M9 MountingHole_2.2mm_M2, Q1 Si7139DP, U1 ATSAMD21G18A-A, U2 MPU-6000, U3 MCF8316A, U4 MCP1826S, U5 MCF8316A, U6 MCF8316A, U7 MCF8316A, U8 TPS62163DSG

Commit message: done?
Parts:
- removed R13: 10k, Resistor_SMD:R_0603_1608Metric_Pad0.98x0.95mm_HandSolder
- removed R16: 100k, Resistor_SMD:R_0603_1608Metric_Pad0.98x0.95mm_HandSolder
- removed U2: MPU-6000, Sensor_Motion:InvenSense_QFN-24_4x4mm_P0.5mm
- added C21: 100nF, Capacitor_SMD:C_0603_1608Metric_Pad1.08x0.95mm_HandSolder, B.Cu at (114.0, 74.3)
- added C22: 22uF, Capacitor_SMD:C_1206_3216Metric_Pad1.33x1.80mm_HandSolder, B.Cu at (116.6, 74.4)
- added C23: 1uF, Capacitor_SMD:C_0603_1608Metric_Pad1.08x0.95mm_HandSolder, F.Cu at (123.0, 77.3)
- added C24: 1uF, Capacitor_SMD:C_0603_1608Metric_Pad1.08x0.95mm_HandSolder, F.Cu at (114.1, 80.3)
- added C25: 1uF, Capacitor_SMD:C_0603_1608Metric_Pad1.08x0.95mm_HandSolder, F.Cu at (115.2, 70.7)
- added C26: 47nF, Capacitor_SMD:C_0603_1608Metric_Pad1.08x0.95mm_HandSolder, F.Cu at (118.3, 72.2)
- added C27: 22uF, Capacitor_SMD:C_1206_3216Metric_Pad1.33x1.80mm_HandSolder, F.Cu at (122.0, 74.0)
- added C28: 100nF, Capacitor_SMD:C_0603_1608Metric_Pad1.08x0.95mm_HandSolder, B.Cu at (113.2, 124.6)
- added C29: 22uF, Capacitor_SMD:C_1206_3216Metric_Pad1.33x1.80mm_HandSolder, B.Cu at (114.2, 121.5)
- added C30: 1uF, Capacitor_SMD:C_0603_1608Metric_Pad1.08x0.95mm_HandSolder, F.Cu at (120.4, 118.2)
- added C31: 1uF, Capacitor_SMD:C_0603_1608Metric_Pad1.08x0.95mm_HandSolder, F.Cu at (118.3, 127.3)
- added C32: 1uF, Capacitor_SMD:C_0603_1608Metric_Pad1.08x0.95mm_HandSolder, F.Cu at (111.0, 121.1)
- added C33: 47nF, Capacitor_SMD:C_0603_1608Metric_Pad1.08x0.95mm_HandSolder, F.Cu at (113.8, 119.4)
- added C34: 22uF, Capacitor_SMD:C_1206_3216Metric_Pad1.33x1.80mm_HandSolder, F.Cu at (117.3, 117.2)
- added C35: 100nF, Capacitor_SMD:C_0603_1608Metric_Pad1.08x0.95mm_HandSolder, B.Cu at (186.4, 125.4)
- added C44: 10nF, Capacitor_SMD:C_0603_1608Metric_Pad1.08x0.95mm_HandSolder, F.Cu at (155.7, 99.2)
- added C45: 2.2uF, Capacitor_SMD:C_0603_1608Metric_Pad1.08x0.95mm_HandSolder, B.Cu at (153.7, 102.6)
- added D1: BZT52H-B12, Diode_SMD:D_SOD-123, B.Cu at (128.7, 86.9)
- added D2: SMAJ18A, Diode_SMD:D_SMA_Handsoldering, F.Cu at (129.0, 90.2)
- added D3: LED_Small, LED_SMD:LED_0402_1005Metric_Pad0.77x0.64mm_HandSolder, F.Cu at (159.9, 97.4)
- added J15: Conn_01x04_Socket, Connector_PinSocket_1.00mm:PinSocket_1x04_P1.00mm_Vertical_SMD_Pin1Left, F.Cu at (146.0, 103.3)
- added L2: 2.2uH, Inductor_SMD:L_1008_2520Metric_Pad1.43x2.20mm_HandSolder, B.Cu at (121.1, 74.6)
- added L3: 2.2uH, Inductor_SMD:L_1008_2520Metric_Pad1.43x2.20mm_HandSolder, B.Cu at (117.3, 118.8)
- added R12: 10k, Resistor_SMD:R_0402_1005Metric_Pad0.72x0.64mm_HandSolder, F.Cu at (121.9, 120.7)
- added R4: 10k, Resistor_SMD:R_0402_1005Metric_Pad0.72x0.64mm_HandSolder, B.Cu at (155.7, 99.1)
- added R9: 10k, Resistor_SMD:R_0402_1005Metric_Pad0.72x0.64mm_HandSolder, F.Cu at (121.5, 80.0)
- added U9: ICM-20602, Package_LGA:LGA-16_3x3mm_P0.5mm, F.Cu at (151.9, 102.1)
- C6: moved to F.Cu
- C8: moved to B.Cu
- C9: value 2.2nF -> 330uF; footprint Capacitor_SMD:C_0603_1608Metric_Pad1.08x0.95mm_HandSolder -> Capacitor_SMD:CP_Elec_10x10.5
- J1: footprint Connector_PinHeader_2.54mm:PinHeader_1x05_P2.54mm_Vertical -> Connector_PinSocket_1.00mm:PinSocket_1x05_P1.00mm_Vertical_SMD_Pin1Left
- R1, R15, R17, R2, R3, R5: footprint Resistor_SMD:R_0603_1608Metric_Pad0.98x0.95mm_HandSolder -> Resistor_SMD:R_0402_1005Metric_Pad0.72x0.64mm_HandSolder
- R6: value 10k -> 220; footprint Resistor_SMD:R_0603_1608Metric_Pad0.98x0.95mm_HandSolder -> Resistor_SMD:R_0402_1005Metric_Pad0.72x0.64mm_HandSolder
- U8: value TPS62163DSG -> TPS62162DSG
- moved R6 27.1 mm to (157.6, 97.4), turned to 180 degrees
- moved C36 20.5 mm to (182.2, 126.8)
- moved C37 20.5 mm to (176.4, 123.0)
- moved C41 20.5 mm to (178.0, 126.1)
- moved L4 20.5 mm to (177.7, 125.7)
- moved R15 20.5 mm to (178.5, 120.0)
- moved C38 20.5 mm to (186.1, 119.1)
- moved C39 20.5 mm to (184.8, 129.6), turned to -29.475 degrees
- moved C40 20.5 mm to (182.0, 127.6)
- moved C9 17.8 mm to (136.1, 97.7), turned to -90 degrees
- moved C7 15.2 mm to (155.3, 102.4), turned to 180 degrees
- moved R17 13.4 mm to (131.7, 88.8), turned to 0 degrees
- moved C6 10.8 mm to (173.9, 101.4), turned to 180 degrees
- moved C8 10.5 mm to (152.2, 102.6), turned to 90 degrees
- moved R2 6.57 mm to (175.6, 92.3), turned to 90 degrees
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- renumbered C10 to C36, C35 to C39
Connections:
- net Net-(U4-VI) renamed +5V
- C37 pad 1: Net-(U3-DVDD) -> Net-(U7-DVDD)
- C38 pad 1: Net-(U3-AVDD) -> Net-(U7-AVDD)
- C39 pad 1: Net-(U3-CP) -> Net-(U7-CP)
- C40 pad 1: Net-(U3-CPH) -> Net-(U7-CPH)
- C40 pad 2: Net-(U3-CPL) -> Net-(U7-CPL)
- C7 pad 1: Net-(U2-REGOUT) -> GND
- C7 pad 2: GND -> Net-(U9-REGOUT)
- C9 pad 1: Net-(U2-CPOUT) -> VBAT
- R15 pad 2: Net-(U3-BRAKE) -> Net-(U7-BRAKE)
- R6 pad 1: Net-(U3-DVDD) -> Net-(D3-K)
- R6 pad 2: DRVOFF_ALL -> GND
- U1 pad 15: /mcu/CRSF_TX -> CRSF_TX
- U1 pad 16: /mcu/CRSF_RX -> CRSF_RX
Routing:
- net VBAT: track 24.1 -> 55.4 mm
- net GND: track 132.3 -> 158.8 mm, vias 43 -> 50
- net +5V: track 9.78 -> 34.9 mm, vias 2 -> 5
- net IMU_INT: track 25.1 -> 7.72 mm, vias 0 -> 2
- net IMU_MISO: track 21.5 -> 5.29 mm, vias 0 -> 2
- net IMU_CS: track 21.3 -> 8.43 mm, vias 0 -> 2
- net Net-(J1-RESET): track 43.7 -> 31.8 mm
- net CRSF_TX: track 0.00 -> 11.3 mm
- net +3V3: track 97.2 -> 86.4 mm
- net IMU_MOSI: track 12.6 -> 3.55 mm, vias 2 -> 0
- net IMU_SCK: track 12.6 -> 3.55 mm, vias 2 -> 0
- net DRVOFF_ALL: track 207.4 -> 198.7 mm, vias 7 -> 5
- net Net-(U3-DVDD): track 11.3 -> 3.47 mm
- net CRSF_RX: track 0.00 -> 7.49 mm
- net Net-(D1-A): track 11.4 -> 3.98 mm
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- added copper zone on F.Cu, net GND

Commit message: done
Parts:
- C19, C20: moved to B.Cu
- C44: footprint Capacitor_SMD:C_0603_1608Metric_Pad1.08x0.95mm_HandSolder -> Capacitor_SMD:C_0402_1005Metric_Pad0.74x0.62mm_HandSolder; moved to B.Cu
- moved C44 6.42 mm to (150.4, 102.9), turned to 90 degrees
- moved C20 3.75 mm to (160.5, 101.9), turned to 90 degrees
- moved C19 3.55 mm to (162.0, 101.9), turned to -90 degrees
- moved C14 0.47 mm to (181.7, 72.2)
- moved C37 0.33 mm to (176.8, 123.1)
Routing:
- net GND: track 158.8 -> 155.3 mm, vias 50 -> 52
- net +3V3: track 86.4 -> 87.3 mm, vias 7 -> 8
- net M4_PWM: track 43.1 -> 43.7 mm
